File: Tempus B.brd (EAGLE design)
At the start: 100 x 34 mm, 37 parts, among them J1 PJ-102A, J2 AVR ISP, J3 GPS, J4 5-1814832-1, U1 ATTINY85-20SU, U2 HT16K33-28SOP, U3 FGPMMOPA6H, U5 DS3231MZ+, U6 L4931CZ33, U7 LM75BIM

Commit message: Tweaking LED resistor values
After testing with the LEDs I ordered, it turns out we need a really
tiny current (0.5mA to 1mA) for the LEDs.
Parts:
- R5: value 470R -> 1K
- R6: value 150R -> 470R
Changed lines of the file:
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@@
 <attribute name="VALUE" x="67.818" y="21.59" size="1.27" layer="27" rot="R180"/>
 </element>
-<element name="R5" library="rcl" package="R1206" value="470R" x="71.628" y="15.24" smashed="yes" rot="R180">
+<element name="R5" library="rcl" package="R1206" value="1K" x="71.628" y="15.24" smashed="yes" rot="R180">
 <attribute name="NAME" x="72.898" y="13.97" size="1.27" layer="25" rot="R180"/>
 <attribute name="VALUE" x="78.232" y="15.748" size="1.27" layer="27" rot="R180"/>
 </element>
-<element name="R6" library="rcl" package="R1206" value="150R" x="71.628" y="19.304" smashed="yes" rot="R180">
+<element name="R6" library="rcl" package="R1206" value="470R" x="71.628" y="19.304" smashed="yes" rot="R180">
 <attribute name="NAME" x="72.898" y="18.034" size="1.27" layer="25" rot="R180"/>
 <attribute name="VALUE" x="78.232" y="19.812" size="1.27" layer="27" rot="R180"/>
